File: Board/TLM-18-Wrap-Up-Supervisor/TLM-18-Wrap-Up-Supervisor.kicad_pcb (KiCad board)
At the start: 2 copper layers, 108 x 68 mm, 24 parts, among them J1 Conn_01x02, J2 DB9_Male, J3 DB9_Female, U1 LM2596T-5, U2 LS7366R, U3 ADM488ANZ, Y1 AB26T-32.000kHZ

Commit message: Updated board SS + BOM
Changed crystal to prepackaged oscillator, added extra silkscreen marks
Parts:
- removed C2, C3: 15pF, Capacitor_THT:C_Rect_L4.0mm_W2.5mm_P2.50mm
- removed R1: 1M, Resistor_THT:R_Axial_DIN0207_L6.3mm_D2.5mm_P7.62mm_Horizontal
- removed Y1: AB26T-32.000kHZ, Crystal:Crystal_DS26_D2.0mm_L6.0mm_Horizontal
- added X1: CXO_DIP8, Oscillator:Oscillator_DIP-8, F.Cu at (105.2, 131.6)
- moved G*** 12.8 mm to (122.4, 110.7)
- moved J2 1.70 mm to (92.1, 107.0)
Connections:
- U2 pad 1: Net-(C3-Pad2) -> unconnected-(U2-Pad1)
Routing:
- net Net-(C3-Pad2): track 15.7 -> 0.00 mm
- net Net-(D2-Pad1): track 0.00 -> 8.66 mm
- net /ENC_Z: track 13.0 -> 11.3 mm
- net /ENC_B: track 13.1 -> 11.4 mm
- net /ENC_A: track 13.2 -> 11.5 mm
- net Net-(U2-Pad2): track 15.0 -> 13.5 mm
- net /CNT_EN: track 86.9 -> 86.1 mm
Other:
- board text added: "COM"
- board text added: "COM Connector Pinout: 1-Z 2-Y 5-SHIELD 6-B 7-A"
- board text added: "ENCODER"
- board text added: "Encoder Connector Pinout: 1-GND 2-Z 3-B 4-A 7-+5V 8-GND"
